File: Sweep v2.2/sweepv2.kicad_pcb (KiCad board)
At the start: 2 copper layers, 216.9 x 86.4 mm, 48 parts, among them J1 AudioJack4dpb, J2 AudioJack4dpb, SW10 SW_Push, SW11 SW_Push, SW11_r1 SW_Push, SW12 SW_Push, SW12_r1 SW_Push, SW13_r1 SW_Push, SW14 SW_Push, SW15 SW_Push, SW15_r1 SW_Push, SW16 SW_Push, SW16_r1 SW_Push, SW17 SW_Push, SW17_r1 SW_Push, SW18 SW_Push, SW18_r1 SW_Push, SW2 SW_Push, SW20 SW_Push, SW20_r1 SW_Push, SW21 SW_Push, SW21_r1 SW_Push, SW2_r1 SW_Push, SW3 SW_Push, SW3_r1 SW_Push, SW4 SW_Push, SW4_r1 SW_Push, SW5 SW_Push, SW5_r1 SW_Push, SW6 SW_Push, SW6_r1 SW_Push, SW7_r1 SW_Push, SW8 SW_Push, SW8_r1 SW_Push, SW9 SW_Push, SW9_r1 SW_Push, U1 ProMicro-kbd, U2 ProMicro-kbd

Commit message: TRRS and Reset removed
Parts:
- removed J1, J2: AudioJack4dpb, Kailh:TRRS-PJ-320A
- removed RSW1, RSW2: SW_Push, kbd:SW_SPST_B3U-1000P
Routing:
- net vcc: track 61.1 -> 0.00 mm, vias 1 -> 0
- net reset_r: track 38.0 -> 0.00 mm, vias 1 -> 0
- net Switch18: track 35.7 -> 0.00 mm, vias 1 -> 0
- net Switch18_r: track 31.1 -> 0.00 mm, vias 1 -> 0
- net reset: track 27.3 -> 0.00 mm, vias 1 -> 0
- net gnd: track 40.7 -> 21.0 mm

Commit message: backside writing changed
Other:
- board text added: "No cat was harmed in the making of this keyboard."
- board text removed: "Sweep is based on the Ferris."
